File: rc-z80ram.sch (KiCad schematic (older format))
At the start: 18 parts, among them J1 Conn_01x39_Male, J2 Conn_01x10_Male, U1 Z80CPU, U2 AS6C1008, U3 DS1233-5, U4 4017, X1 7.3728MHz

Commit message: Move components, clean up routing
Move components in order to shorten and neaten clock traces. Make jumpers easier to reach, move oscillator to bottom of card to reduce shorting risk.
Parts:
- J1: value Conn_01x39_Male -> RC2014
- J2: value Conn_01x10_Male -> RC2014_Enh
Connections:
- net CDIV: now also U4.2 (Q1); no longer U4.3 (Q0)
- net CLK: now also JP3.2; no longer JP3.1
- net OSC: now also JP3.1; no longer JP3.2
Other:
- moved on the sheet: C1, C2, C3, C4, C5, JP1, JP2, JP3, JP4, JP5, RN1, U1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

Commit message: Add BOM, tidy up schematic
Parts:
- JP3: symbol Device:Jumper_NC_Small -> Jumper:Jumper_2_Open
- U1: value Z80CPU -> Z84C0008
- U4: value 4017 -> CD74HC4017
Other:
- moved on the sheet: J2
